File: eagle/watchplb.brd (EAGLE design)
At the start: 100 x 100 mm, 224 parts, among them IC1 SAM-M8Q, IC2 BM70BLES1FC2-0B03AA, IC3 LM1117DTX-ADJ-12V, IC5 LM1117DTX-ADJ-10V, IC6 LM1117DTX-ADJ-3V3, J3 BNCPTH, Q1 8MHz / LFXTAL020423Reel, Q2 BC817-25SMD, Q3 DMN3023L-7, Q4 16MHz_LFXTAL051370Reel, Q5 CSD18534Q5A, Q6 CSD18534Q5A, Q7 DMN3023L-7, U1 MCP111-XXXXX/TO, U2 STM32L073RZ, U3 MCP2200-I/SS, U4 TPD3E001DRLR, U5 BQ7790504

Commit message: added some datasheets and continued with layout
Parts:
- removed C50: 4.7uF, resistor:C0805K
- removed VIBR: PTR1B2,54, testpad:B2,54
- added BAT_PACK_POS, USB_DN, USB_DP, USB_ID: PTR1B2,54, testpad:B2,54
- added C63: 4.7uF low esr 80-T521B475M35ATE150, rcl:B/3528-21R
- R50: device resistor:M0805 -> resistor:R2512
- moved RF_SIGNAL 597.0 mm to (88.1, 89.6)
- moved BAT_ADC 518.1 mm to (-20.7, 89.8)
- moved R61 517.6 mm to (-20.7, 96.2)
- moved R60 517.3 mm to (-18.6, 100.1)
- moved C52 481.7 mm to (6.55, 70.0), turned to 180 degrees
- moved C62 478.9 mm to (-101.5, 140.2), turned to 90 degrees
- moved D10 476.6 mm to (7.01, 53.8)
- moved SPI2_IRQ 471.6 mm to (129.5, 40.1), turned to 180 degrees
- moved C51 469.2 mm to (6.55, 61.6), turned to 180 degrees
- moved SPI2_MOSI 466.6 mm to (125.9, 40.8), turned to 180 degrees
- moved R52 465.3 mm to (25.5, 39.2), turned to 180 degrees
- moved J4 463.7 mm to (1.98, 31.5)
- moved SPI2_MISO 462.9 mm to (123.6, 41.5), turned to 180 degrees
- moved SPI2_CLK 460.7 mm to (122.7, 42.7), turned to 180 degrees
- moved R50 460.6 mm to (26.5, 44.7), turned to 90 degrees
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Connections:
- net N$41 renamed ANT_N
- net N$44 renamed ANT_P
- removed net N$75: C50.1, D10.A, L8.4
- new net N$87: J4.ID, USB_ID.TP
- new net N$88: J4.D+, USB_DP.TP
- new net N$90: J4.D-, USB_DN.TP
- new net N$91: C63.-, D10.A, L8.3
- net BAT_PACK_POS: now also BAT_PACK_POS.TP
- net IND_LED_B: now also U2.26; no longer U2.27
- net IND_LED_G: now also U2.25; no longer U2.28
- net IND_LED_R: now also U2.28; no longer U2.25
- net IND_LED_W: now also U2.27; no longer U2.26
- net N$61: now also C63.+; no longer C50.2
- net N$70: now also L8.4; no longer L8.3
- net POW_LED_G2: now also U2.21; no longer U2.23
- net POW_LED_G3: now also U2.20; no longer U2.24
- net POW_LED_R: now also U2.24; no longer U2.20
- net POW_LED_Y: now also U2.23; no longer U2.21
- net VIBRATOR: no longer VIBR.TP
Routing:
- net GND: track 222.0 -> 600.0 mm, vias 4 -> 18
- net +3V3: track 149.2 -> 328.8 mm, vias 0 -> 1
- net N$84: track 9.65 -> 106.7 mm, vias 0 -> 1
- net N$69: track 0.00 -> 59.9 mm
- net +12V: track 17.4 -> 76.4 mm
- net BT_HCI_TXD: track 0.00 -> 51.1 mm
- net INT_POWER: track 0.00 -> 47.0 mm, vias 0 -> 3
- net BT_HCI_RXD: track 0.00 -> 42.9 mm
- net BAT_PACK_POS: track 15.2 -> 52.3 mm
- net V+STM: track 0.00 -> 35.6 mm
- net BT_P2_0_MODE: track 0.00 -> 33.5 mm, vias 0 -> 1
- net N$74: track 0.00 -> 31.9 mm, vias 0 -> 2
- net BT_NRST: track 0.00 -> 28.6 mm, vias 0 -> 1
- net N$77: track 0.00 -> 28.5 mm, vias 0 -> 2
- net N$37: track 0.00 -> 27.5 mm
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- added copper zone on layer 16, net GND

Commit message: continued layout
Parts:
- moved B2 361.4 mm to (193.9, -65.1)
- moved C1 361.4 mm to (194.0, -46.9)
- moved C2 361.4 mm to (194.0, -53.2)
- moved C3 361.4 mm to (194.0, -59.6)
- moved C62 361.4 mm to (193.2, -68.9)
- moved GPS_EXTINT 361.4 mm to (198.9, -44.2)
- moved GPS_NRESET 361.4 mm to (198.9, -37.9)
- moved GPS_RX 361.4 mm to (198.9, -63.2)
- moved GPS_SCL 361.4 mm to (198.9, -57.0)
- moved GPS_SDA 361.4 mm to (198.9, -50.6)
- moved GPS_TX 361.4 mm to (198.9, -69.6)
- moved IC1 361.4 mm to (176.8, -55.5)
- moved R1 361.4 mm to (188.5, -53.8)
- moved R2 361.4 mm to (188.4, -58.8)
- moved BTN_2 144.0 mm to (79.2, 7.32)
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Connections:
- removed net GND1: LED4.C
- removed net GND2: LED5.C
- net GND: now also LED4.C, LED5.C
Routing:
- net SPI2_CLK: track 24.4 -> 110.1 mm, vias 0 -> 3
- net BT_HCI_RXD: track 42.9 -> 118.4 mm, vias 0 -> 2
- net GND: track 600.0 -> 675.1 mm, vias 18 -> 19
- net SPI2_IRQ: track 18.6 -> 92.0 mm, vias 0 -> 2
- net SPI2_MOSI: track 19.7 -> 87.6 mm, vias 0 -> 3
- net BT_HCI_TXD: track 51.1 -> 116.9 mm, vias 0 -> 2
- net SPI2_SEL_RFTX: track 26.0 -> 89.8 mm, vias 0 -> 2
- net SPI2_MISO: track 22.9 -> 83.0 mm, vias 0 -> 3
- net +3V3: track 328.8 -> 388.1 mm
- net BAT_PACK_POS: track 52.3 -> 102.9 mm
- net N$37: track 27.5 -> 69.2 mm
- net IND_LED_R: track 0.00 -> 39.0 mm
- net IND_LED_W: track 0.00 -> 37.4 mm
- net IND_LED_B: track 0.00 -> 35.9 mm
- net IND_LED_G: track 0.00 -> 34.4 mm
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