File: eagle/watchplb.brd (EAGLE design)
At the start: 100 x 100 mm, 227 parts, among them IC1 SAM-M8Q, IC2 BM70BLES1FC2-0B03AA, IC3 LM1117DTX-ADJ-12V, IC5 LM1117DTX-ADJ-10V, IC6 LM1117DTX-ADJ-3V3, J3 BNCPTH, Q1 8MHz / LFXTAL020423Reel, Q2 BC817-25SMD, Q3 DMN3023L-7, Q4 16MHz_LFXTAL051370Reel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

Commit message: continued layout
Parts:
- added JP4, JP5: (no value), pinhead:1X08
- moved NRST_MCU 111.3 mm to (74.1, 43.1)
- moved SWD_RXD 105.2 mm to (54.9, 35.7)
- moved GPS_EXTINT 98.6 mm to (166.9, 49.1)
- moved GPS_NRESET 98.6 mm to (166.9, 55.3)
- moved GPS_RX 98.6 mm to (166.9, 30.0)
- moved GPS_SCL 98.6 mm to (166.9, 36.3)
- moved GPS_SDA 98.6 mm to (166.9, 42.7)
- moved GPS_TX 98.6 mm to (166.9, 23.6)
- moved B2 98.6 mm to (161.8, 28.2)
- moved C1 98.6 mm to (162.0, 46.3)
- moved C2 98.6 mm to (162.0, 40.1)
- moved C3 98.6 mm to (162.0, 33.7)
- moved C62 98.6 mm to (161.2, 24.4)
- moved IC1 98.6 mm to (144.8, 37.8)
- moved R1 98.6 mm to (156.5, 39.5)
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Connections:
- net +3V3: now also JP4.1, JP5.1
- net GND: now also JP4.2, JP5.2
- net GPS_EXTINT: now also JP4.5, JP5.5
- net GPS_NRESET: now also JP4.6, JP5.6
- net GPS_RXD: now also JP4.7, JP5.7
- net GPS_SCL: now also JP4.3, JP5.3
- net GPS_SDA: now also JP4.4, JP5.4
- net GPS_TXD: now also JP4.8, JP5.8
Routing:
- net +3V3: track 388.1 -> 487.1 mm, vias 1 -> 6
- net GND: track 675.1 -> 728.3 mm, vias 19 -> 28
- net GPS_SCL: track 0.00 -> 51.8 mm
- net GPS_SDA: track 0.00 -> 51.5 mm
- net GPS_EXTINT: track 0.00 -> 51.2 mm
- net GPS_NRESET: track 0.00 -> 50.9 mm
- net NRST: track 24.5 -> 67.4 mm, vias 0 -> 3
- net SWDIO: track 0.00 -> 33.7 mm, vias 0 -> 2
- net GPS_TXD: track 0.00 -> 32.2 mm
- net GPS_RXD: track 0.00 -> 30.7 mm
- net SWDCLK: track 0.00 -> 28.8 mm, vias 0 -> 2
- net BTN_4: track 22.8 -> 50.9 mm, vias 0 -> 2
- net MCU_WAKEUP: track 29.6 -> 9.75 mm
- net BTN_3: track 37.2 -> 55.5 mm, vias 0 -> 2
- net BAT_ADC: track 0.00 -> 16.5 mm
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
Commit message: layout v1 fertig
Parts:
- removed GPS_EXTINT, GPS_NRESET, GPS_RX, GPS_SCL, GPS_SDA, GPS_TX: PTR1B2,54, testpad:B2,54
- C62: device resistor:C0805K -> resistor:C0805
- moved JP5 51.5 mm to (152.1, 21.9)
- moved IC1 34.8 mm to (176.5, 23.5)
- moved R1 34.6 mm to (185.5, 20.6), turned to 90 degrees
- moved R2 30.4 mm to (178.3, 13.4), turned to 90 degrees
- moved C1 22.3 mm to (179.4, 32.3)
- moved B2 21.0 mm to (175.3, 12.0), turned to 180 degrees
- moved C2 18.5 mm to (167.5, 22.4), turned to 270 degrees
- moved C62 15.7 mm to (172.5, 13.4)
- moved Q1 11.6 mm to (81.0, 47.1), turned to 315 degrees
- moved C3 9.14 mm to (167.5, 26.4), turned to 90 degrees
- moved C14 0.91 mm to (70.6, 48.6)
- moved C15 0.91 mm to (66.4, 48.6)
- moved R9 0.91 mm to (66.4, 46.5)
- moved C10 0.76 mm to (66.4, 44.2)
- moved R54 0.61 mm to (64.9, 97.5)
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Connections:
- net GPS_EXTINT: no longer GPS_EXTINT.TP
- net GPS_NRESET: no longer GPS_NRESET.TP
- net GPS_RXD: no longer GPS_RX.TP
- net GPS_SCL: no longer GPS_SCL.TP
- net GPS_SDA: no longer GPS_SDA.TP
- net GPS_TXD: no longer GPS_TX.TP
Routing:
- net CHARGER_SS: track 0.00 -> 119.9 mm, vias 0 -> 1
- net BAT_ADC: track 16.5 -> 118.4 mm, vias 0 -> 3
- net CHARGER_CH_PRECH: track 0.00 -> 85.4 mm, vias 0 -> 2
- net MCU_WAKEUP: track 9.75 -> 83.3 mm, vias 0 -> 2
- net VIBRATOR: track 4.37 -> 72.8 mm, vias 0 -> 2
- net +3V3: track 487.1 -> 549.8 mm, vias 6 -> 9
- net NRST: track 67.4 -> 127.0 mm, vias 3 -> 4
- net GPS_SCL: track 51.8 -> 103.6 mm, vias 0 -> 1
- net GPS_TXD: track 32.2 -> 82.0 mm
- net GPS_RXD: track 30.7 -> 76.7 mm
- net N$79: track 0.00 -> 41.7 mm
- net GPS_SDA: track 51.5 -> 85.8 mm, vias 0 -> 1
- net GPS_NRESET: track 50.9 -> 84.3 mm
- net GPS_EXTINT: track 51.2 -> 83.0 mm
- net GND: track 728.3 -> 698.1 mm, vias 28 -> 59
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- added copper zone on layer 1, net GND
Other:
- board size 100 x 100 mm -> 200 x 100 mm

Commit message: added text and fh logo
Parts:
- removed JP1: SWD, pinhead:1X05
- added PR0>: SWD, pinhead:1X05
- added U$4: (no value), Hick:FH_LOGO
- moved SPI2_CLK 0.68 mm to (31.5, 19.2)
- moved FB1 0.61 mm to (9.14, 22.9)
- renumbered JP4 to GPS>, JP5 to <GPS
Connections:
- removed net USB_DATA_NEG: J2.D-, U4.1
- removed net USB_DATA_POS: J2.D+, R27.2, U4.2
- new net USB_DATA_N: J2.D-, U2.44, U4.1
- new net USB_DATA_P: J2.D+, R27.2, U2.45, U4.2
- net +3V3: now also PR0>.4; no longer JP1.4
- net GND: now also PR0>.1; no longer JP1.1
- net NRST: now also PR0>.5; no longer JP1.5
- net SWDCLK: now also PR0>.3; no longer JP1.3
- net SWDIO: now also PR0>.2; no longer JP1.2
- net VIBRATOR: now also U2.50; no longer U2.44
Routing:
- net USB_DATA_N: track 0.00 -> 80.8 mm, vias 0 -> 4
- net USB_DATA_P: track 0.00 -> 80.7 mm, vias 0 -> 4
- net VIBRATOR: track 72.8 -> 83.3 mm
- net GND: track 698.1 -> 706.4 mm, vias 59 -> 161
- net USB_DATA_POS: track 7.99 -> 0.00 mm
- net NRST: track 127.0 -> 132.3 mm
- net +5V: track 38.2 -> 42.4 mm
- net USB_DATA_NEG: track 4.04 -> 0.00 mm
- net +3V3: track 549.8 -> 552.3 mm
- net SWDCLK: track 28.8 -> 29.7 mm
- net SPI2_CLK: track 104.4 -> 103.8 mm
Other:
- board text added: "Charge"
- board text added: "FTDI"
- board text added: "NRST 3V3 SWDCLK SWDIO GND"
- board text added: "Native"
- board text added: "WatchPLB Mainboard V1.0 c by Samuel Hick, HSD 2018 Made in Austria"
