File: eagle/watchplb.sch (EAGLE design)
At the start: 227 parts, among them IC1 SAM-M8Q, IC2 BM70BLES1FC2-0B03AA, IC3 LM1117DTX-ADJ-12V, IC5 LM1117DTX-ADJ-10V, IC6 LM1117DTX-ADJ-3V3, J3 BNCPTH, Q1 8MHz / LFXTAL020423Reel, Q2 BC817-25SMD, Q3 DMN3023L-7, Q4 16MHz_LFXTAL051370Reel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

Commit message: continued layout
Connections:
- removed net GND1: LED4.C
- removed net GND2: LED5.C
- net GND: now also LED4.C, LED5.C
Changed lines of the file:
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@@
 <wire x1="134.62" y1="38.1" x2="132.08" y2="38.1" width="0.1524" layer="91"/>
 <junction x="134.62" y="48.26"/>
+<pinref part="LED5" gate="G$1" pin="C"/>
+<wire x1="132.08" y1="17.78" x2="134.62" y2="17.78" width="0.1524" layer="91"/>
+<wire x1="134.62" y1="17.78" x2="134.62" y2="27.94" width="0.1524" layer="91"/>
+<junction x="134.62" y="38.1"/>
+<pinref part="LED4" gate="G$1" pin="C"/>
+<wire x1="134.62" y1="27.94" x2="134.62" y2="38.1" width="0.1524" layer="91"/>
+<wire x1="132.08" y1="27.94" x2="134.62" y2="27.94" width="0.1524" layer="91"/>
+<junction x="134.62" y="27.94"/>
 </segment>
 <segment>
@@
 </segment>
 </net>
-<net name="GND1" class="0">
-<segment>
-<pinref part="LED4" gate="G$1" pin="C"/>
-<wire x1="134.62" y1="38.1" x2="134.62" y2="27.94" width="0.1524" layer="91"/>
-<wire x1="134.62" y1="27.94" x2="132.08" y2="27.94" width="0.1524" layer="91"/>
-</segment>
-</net>
 <net name="N$12" class="0">
 <segment>
@@
 </segment>
 </net>
-<net name="GND2" class="0">
-<segment>
-<pinref part="LED5" gate="G$1" pin="C"/>
-<wire x1="134.62" y1="27.94" x2="134.62" y2="17.78" width="0.1524" layer="91"/>
-<wire x1="134.62" y1="17.78" x2="132.08" y2="17.78" width="0.1524" layer="91"/>
-</segment>
-</net>
 <net name="N$16" class="0">
 <segment>
@@
 <segment>
 <pinref part="R15" gate="G$1" pin="2"/>
-<wire x1="111.76" y1="17.78" x2="86.36" y2="7.62" width="0.1524" layer="91"/>
-<wire x1="86.36" y1="7.62" x2="86.36" y2="71.12" width="0.1524" layer="91"/>
+<wire x1="111.76" y1="17.78" x2="86.36" y2="17.78" width="0.1524" layer="91"/>
+<wire x1="86.36" y1="17.78" x2="86.36" y2="71.12" width="0.1524" layer="91"/>
 <label x="96.52" y="73.66" size="1.778" layer="95"/>
 <pinref part="U2" gate="A" pin="PB2"/>

Commit message: continued layout
Parts:
- added JP4, JP5: (no value), pinhead:PINHD-1X8
Connections:
- net +3V3: now also JP4.1, JP5.1
- net GND: now also JP4.2, JP5.2
- net GPS_EXTINT: now also JP4.5, JP5.5
- net GPS_NRESET: now also JP4.6, JP5.6
- net GPS_RXD: now also JP4.7, JP5.7
- net GPS_SCL: now also JP4.3, JP5.3
- net GPS_SDA: now also JP4.4, JP5.4
- net GPS_TXD: now also JP4.8, JP5.8
Changed lines of the file:
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@@
 <part name="USB_DN" library="testpad" deviceset="PTR1" device="B2,54"/>
 <part name="C63" library="rcl" deviceset="CPOL-EU" device="B/3528-21R" value="4.7uF low esr 80-T521B475M35ATE150 "/>
+<part name="JP4" library="pinhead" deviceset="PINHD-1X8" device=""/>
+<part name="JP5" library="pinhead" deviceset="PINHD-1X8" device=""/>
 </parts>
 <sheets>
@@
 </instance>
 <instance part="C63" gate="G$1" x="403.86" y="261.62" rot="R90"/>
+<instance part="JP4" gate="A" x="584.2" y="142.24"/>
+<instance part="JP5" gate="A" x="594.36" y="142.24"/>
 </instances>
 <busses>
@@
 <pinref part="+3V5" gate="G$1" pin="+3V3"/>
 </segment>
+<segment>
+<pinref part="JP4" gate="A" pin="1"/>
+<pinref part="JP5" gate="A" pin="1"/>
+<wire x1="581.66" y1="152.4" x2="591.82" y2="152.4" width="0.1524" layer="91"/>
+<wire x1="591.82" y1="152.4" x2="609.6" y2="152.4" width="0.1524" layer="91"/>
+<junction x="591.82" y="152.4"/>
+<label x="596.9" y="152.4" size="1.778" layer="95"/>
+</segment>
 </net>
 <net name="GPS_RXD" class="0">
@@
 <pinref part="GPS_RX" gate="G$1" pin="TP"/>
 </segment>
+<segment>
+<pinref part="JP4" gate="A" pin="7"/>
+<pinref part="JP5" gate="A" pin="7"/>
+<wire x1="581.66" y1="137.16" x2="591.82" y2="137.16" width="0.1524" layer="91"/>
+<wire x1="591.82" y1="137.16" x2="609.6" y2="137.16" width="0.1524" layer="91"/>
+<junction x="591.82" y="137.16"/>
+<label x="596.9" y="137.16" size="1.778" layer="95"/>
+</segment>
 </net>
 <net name="GPS_TXD" class="0">
@@
 <pinref part="GPS_TX" gate="G$1" pin="TP"/>
 </segment>
+<segment>
+<pinref part="JP4" gate="A" pin="8"/>
+<pinref part="JP5" gate="A" pin="8"/>
+<wire x1="581.66" y1="134.62" x2="591.82" y2="134.62" width="0.1524" layer="91"/>
+<wire x1="591.82" y1="134.62" x2="609.6" y2="134.62" width="0.1524" layer="91"/>
+<junction x="591.82" y="134.62"/>
+<label x="596.9" y="134.62" size="1.778" layer="95"/>
+</segment>
 </net>
 <net name="GPS_SCL" class="0">
@@
 <label x="175.26" y="66.04" size="1.778" layer="95"/>
 <pinref part="GPS_SCL" gate="G$1" pin="TP"/>
+</segment>
+<segment>
+<pinref part="JP4" gate="A" pin="3"/>
+<pinref part="JP5" gate="A" pin="3"/>
+<wire x1="581.66" y1="147.32" x2="591.82" y2="147.32" width="0.1524" layer="91"/>
+<wire x1="591.82" y1="147.32" x2="609.6" y2="147.32" width="0.1524" layer="91"/>
+<junction x="591.82" y="147.32"/>
+<label x="596.9" y="147.32" size="1.778" layer="95"/>
 </segment>
 </net>
@@
 <pinref part="GPS_SDA" gate="G$1" pin="TP"/>
 </segment>
+<segment>
+<pinref part="JP4" gate="A" pin="4"/>
+<pinref part="JP5" gate="A" pin="4"/>
+<wire x1="581.66" y1="144.78" x2="591.82" y2="144.78" width="0.1524" layer="91"/>
+<wire x1="591.82" y1="144.78" x2="609.6" y2="144.78" width="0.1524" layer="91"/>
+<junction x="591.82" y="144.78"/>
+<label x="596.9" y="144.78" size="1.778" layer="95"/>
+</segment>
 </net>
 <net name="GPS_EXTINT" class="0">
@@
 <pinref part="GPS_EXTINT" gate="G$1" pin="TP"/>
 </segment>
+<segment>
+<pinref part="JP4" gate="A" pin="5"/>
+<pinref part="JP5" gate="A" pin="5"/>
+<wire x1="581.66" y1="142.24" x2="591.82" y2="142.24" width="0.1524" layer="91"/>
+<wire x1="591.82" y1="142.24" x2="609.6" y2="142.24" width="0.1524" layer="91"/>
+<junction x="591.82" y="142.24"/>
+<label x="596.9" y="142.24" size="1.778" layer="95"/>
+</segment>
 </net>
 <net name="GPS_NRESET" class="0">
@@
 <label x="175.26" y="73.66" size="1.778" layer="95"/>
 <pinref part="GPS_NRESET" gate="G$1" pin="TP"/>
+</segment>
+<segment>
+<pinref part="JP4" gate="A" pin="6"/>
+<pinref part="JP5" gate="A" pin="6"/>
+<wire x1="581.66" y1="139.7" x2="591.82" y2="139.7" width="0.1524" layer="91"/>
+<wire x1="591.82" y1="139.7" x2="609.6" y2="139.7" width="0.1524" layer="91"/>
+<junction x="591.82" y="139.7"/>
+<label x="596.9" y="139.7" size="1.778" layer="95"/>
 </segment>
 </net>
@@
 <wire x1="292.1" y1="320.04" x2="292.1" y2="322.58" width="0.1524" layer="91"/>
 </segment>
+<segment>
+<pinref part="JP4" gate="A" pin="2"/>
+<pinref part="JP5" gate="A" pin="2"/>
+<wire x1="581.66" y1="149.86" x2="591.82" y2="149.86" width="0.1524" layer="91"/>
+<wire x1="591.82" y1="149.86" x2="609.6" y2="149.86" width="0.1524" layer="91"/>
+<junction x="591.82" y="149.86"/>
+<label x="596.9" y="149.86" size="1.778" layer="95"/>
+</segment>
 </net>

Commit message: layout v1 fertig
Parts:
- removed GPS_EXTINT, GPS_NRESET, GPS_RX, GPS_SCL, GPS_SDA, GPS_TX: PTR1B2,54, testpad:PTR1B2,54
- C62: device resistor:C-EUC0805K -> resistor:C-EUC0805
Connections:
- net GPS_EXTINT: no longer GPS_EXTINT.TP
- net GPS_NRESET: no longer GPS_NRESET.TP
- net GPS_RXD: no longer GPS_RX.TP
- net GPS_SCL: no longer GPS_SCL.TP
- net GPS_SDA: no longer GPS_SDA.TP
- net GPS_TXD: no longer GPS_TX.TP

Commit message: added text and fh logo
Parts:
- renumbered JP1 to PR0>, JP4 to GPS>, JP5 to <GPS
Connections:
- removed net USB_DATA_NEG: J2.D-, U4.IO1
- removed net USB_DATA_POS: J2.D+, R27.2, U4.IO2
- new net USB_DATA_N: J2.D-, U2.PA11, U4.IO1
- new net USB_DATA_P: J2.D+, R27.2, U2.PA12, U4.IO2
- net VIBRATOR: now also U2.PA15; no longer U2.PA11
