File: eagle/Mainboard/watchplb_mainboard_v1_1.sch (EAGLE design)
At the start: 223 parts, among them IC1 SAM-M8Q, IC2 BM70BLES1FC2-0B03AA, IC3 LM1117DTX-ADJ-12V, IC5 LM1117DTX-ADJ-10V, IC6 LM1117DTX-ADJ-3V3, J3 BNCPTH, Q1 8MHz / LFXTAL020423Reel, Q2 BC817-25SMD, Q3 DMN3023L-7, Q4 16MHz_LFXTAL051370Reel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

Commit message: changes requested by armin brandl
Parts:
- removed <GPS: (no value), pinhead:PINHD-1X8
- removed B2: BLM18KG601SN1D, PCB4_Demoboard:B-EU_B0603
- removed C1, C2, C3: 1uF, resistor:C-EUC0805
- removed C62: 4.7uF, resistor:C-EUC0805
- removed IC1: SAM-M8Q, ubloxLib:SAM-M8Q
- removed R1, R2: 47k, resistor:R-EU_M0805
- 3V3, BAT_ADC, BTN_1, BTN_2, BTN_3, BTN_4, BTN_NRST, BT_RX, BT_TX, NRST_MCU, RF_SYSCLK, SPI2_CLK, SPI2_IRQ, SPI2_MISO, SPI2_MOSI, SPI2_SEL_RFTX, SWD_RXD, SWD_TXD, USB_DN, USB_DP, USB_ID: value PTR1B2,54 -> PTR1B1,27; device testpad:PTR1B2,54 -> testpad:PTR1B1,27
Connections:
- removed net N$79: B2.2, C1.1, C2.1, C3.1, C62.1, IC1.VCC, IC1.VCC_IO, IC1.V_BCKP
- net +3V3: no longer <GPS.1, B2.1, R1.1, R2.1
- net GND: no longer <GPS.2, C1.2, C2.2, C3.2, C62.2, IC1.GND
- net GPS_EXTINT: no longer <GPS.5, IC1.EXTINT
- net GPS_NRESET: no longer <GPS.6, IC1.RESET_N
- net GPS_RXD: no longer <GPS.7, IC1.RXD
- net GPS_SCL: no longer <GPS.3, IC1.SCL, R1.2
- net GPS_SDA: no longer <GPS.4, IC1.SDA, R2.2
- net GPS_TXD: no longer <GPS.8, IC1.TXD
Other:
- note removed: "Module alone on this side, check Hardware Integration manual for Layout Suggestions"
- note removed: "SAM-M8Q"
- note removed: "devboard uses 4.7 uF, so i added one of those"
- note removed: "value of caps guessed, not specified in datasheet"
- moved on the sheet: B3, B4, CONFIG_INTERFACE_TEST_POINT, GPS>, IC2, LED1, R3, U1
