File: eagle/Mainboard/watchplb_mainboard_v1_1.brd (EAGLE design)
At the start: 200 x 100 mm, 224 parts, among them IC1 SAM-M8Q, IC2 BM70BLES1FC2-0B03AA, IC3 LM1117DTX-ADJ-12V, IC5 LM1117DTX-ADJ-10V, IC6 LM1117DTX-ADJ-3V3, J3 BNCPTH, Q1 8MHz / LFXTAL020423Reel, Q2 BC817-25SMD, Q3 DMN3023L-7, Q4 16MHz_LFXTAL051370Reel, Q5 CSD18534Q5A, Q6 CSD18534Q5A, Q7 DMN3023L-7, U1 MCP111-XXXXX/TO, U2 STM32L073RZ, U3 MCP2200-I/SS, U4 TPD3E001DRLR, U5 BQ7790504

Commit message: changes requested by armin brandl
Parts:
- removed <GPS: (no value), pinhead:1X08
- removed B2: BLM18KG601SN1D, PCB4_Demoboard:L0603
- removed C1, C2, C3: 1uF, resistor:C0805
- removed C62: 4.7uF, resistor:C0805
- removed IC1: SAM-M8Q, ubloxLib:SAM-M8Q
- removed R1, R2: 47k, resistor:M0805
- added U$5: (no value), watchplb_mainboard_v1_1:FH_LOGO_050
- 3V3, BAT_ADC, BTN_1, BTN_2, BTN_3, BTN_4, BTN_NRST, BT_RX, BT_TX, NRST_MCU, RF_SYSCLK, SPI2_CLK, SPI2_IRQ, SPI2_MISO, SPI2_MOSI, SPI2_SEL_RFTX, SWD_RXD, SWD_TXD, USB_DN, USB_DP, USB_ID: value PTR1B2,54 -> PTR1B1,27; device testpad:B2,54 -> testpad:B1,27
- moved U$4 71.6 mm to (27.7, 81.4), turned to 270 degrees
Connections:
- removed net N$79: B2.2, C1.1, C2.1, C3.1, C62.1, IC1.17, IC1.2, IC1.3
- net +3V3: no longer <GPS.1, B2.1, R1.1, R2.1
- net GND: no longer <GPS.2, C1.2, C2.2, C3.2, C62.2, IC1.1, IC1.10, IC1.11, IC1.15, IC1.16, IC1.20, IC1.4, IC1.5, IC1.6
- net GPS_EXTINT: no longer <GPS.5, IC1.19
- net GPS_NRESET: no longer <GPS.6, IC1.18
- net GPS_RXD: no longer <GPS.7, IC1.14
- net GPS_SCL: no longer <GPS.3, IC1.12, R1.2
- net GPS_SDA: no longer <GPS.4, IC1.9, R2.2
- net GPS_TXD: no longer <GPS.8, IC1.13
Routing:
- net GPS_TXD: track 82.0 -> 32.2 mm
- net GPS_SCL: track 103.6 -> 54.6 mm, vias 1 -> 0
- net GPS_RXD: track 76.7 -> 30.7 mm
- net +3V3: track 552.3 -> 510.5 mm
- net N$79: track 41.7 -> 0.00 mm
- net GPS_SDA: track 85.8 -> 54.4 mm, vias 1 -> 0
- net GPS_NRESET: track 84.3 -> 53.6 mm
- net GPS_EXTINT: track 83.0 -> 54.1 mm
- net GND: track 706.4 -> 686.1 mm, vias 161 -> 1036
- net BTN_1: track 79.1 -> 93.5 mm
Other:
- board size 200 x 100 mm -> 100 x 100 mm
- board text added: "WPLB Main V1_1"

Commit message: weitere Änderungen von Armin Brandl
Routing:
- net GND: track 686.1 -> 671.5 mm, vias 1036 -> 422
