File: eagle/Mainboard/watchplb_mainboard_v1_0.brd (EAGLE design)
At the start: 100 x 100 mm, 216 parts, among them IC2 BM70BLES1FC2-0B03AA, IC3 LM1117DTX-ADJ-12V, IC5 LM1117DTX-ADJ-10V, IC6 LM1117DTX-ADJ-3V3, J3 BNCPTH, Q1 8MHz / LFXTAL020423Reel, Q2 BC817-25SMD, Q3 DMN3023L-7, Q4 16MHz_LFXTAL051370Reel, Q5 CSD18534Q5A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

Commit message: Änderungen laut Besprechung mit Armin (soweit ich mich erinnern kann, ist schon ne woche her)
Parts:
- BAT_PACK_POS: value PTR1B2,54 -> PTR1B1,27; device testpad:B2,54 -> testpad:B1,27
- moved BTN_NRST 1.52 mm to (33.7, 3.66)
- moved RF_SYSCLK 1.02 mm to (33.8, 34.3)
- moved BAT_PACK_POS 0.76 mm to (3.05, 65.7)
- moved C23 0.61 mm to (69.2, 64.5)
- moved C27 0.61 mm to (71.3, 64.5)
- renumbered U$1 to IC4, U$3 to IC1
Routing:
- net GND: track 671.5 -> 183.3 mm, vias 422 -> 399
- net BTN_1: track 93.5 -> 78.5 mm
- net +12V: track 96.3 -> 82.0 mm
- net +3V3: track 510.5 -> 497.5 mm
- net NRST: track 132.3 -> 124.8 mm
- net N$84: track 109.0 -> 103.5 mm
- net N$74: track 31.9 -> 26.5 mm
- net SPI2_MOSI: track 89.5 -> 85.5 mm
- net INT_POWER: track 53.1 -> 56.8 mm
- net USB_DATA_P: track 80.7 -> 77.9 mm
- net SPI2_IRQ: track 92.7 -> 90.1 mm
- net CHARGER_SS: track 119.9 -> 117.5 mm
- net N$80: track 13.5 -> 11.3 mm
- net GPS_SCL: track 54.6 -> 52.4 mm
- net BAT_PACK_POS: track 98.8 -> 96.7 mm
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Other:
- board text added: "WPLB Main V1_0"
- board text removed: "WPLB Main V1_1"

Commit message: kleine Änderungen laut email mit  Armin, veraltete Dateien entfernt, gerber generiert
Parts:
- moved USB_DN 1.59 mm to (18.4, 35.1)
- moved C29 0.48 mm to (81.2, 69.5)
- moved L7 0.39 mm to (84.0, 89.7)
- moved C30 0.34 mm to (84.7, 69.5)
- moved C34 0.34 mm to (81.1, 81.1)
- moved C31 0.30 mm to (82.0, 75.9)
- moved C32 0.30 mm to (81.1, 79.1)
- moved C33 0.30 mm to (84.7, 79.1)
- moved L1 0.30 mm to (82.1, 72.2)
- moved L5 0.30 mm to (84.9, 81.1)
Routing:
- net INT_POWER: track 56.8 -> 51.9 mm
- net ANT_N: track 16.6 -> 14.9 mm
- net N$90: track 16.5 -> 14.9 mm
- net ANT_P: track 17.3 -> 15.7 mm
- net RF_SIGNAL: track 25.3 -> 26.4 mm
- net N$85: track 23.3 -> 22.6 mm
- net N$43: track 7.19 -> 6.53 mm
- net BAT_PACK_GND: track 62.2 -> 61.7 mm
- net N$84: track 103.5 -> 104.0 mm
- net GND: track 183.3 -> 183.5 mm, vias 399 -> 417

Commit message: started BOM
Parts:
- C28, C31: value (none) -> 7.5pF
- C29, C30: value (none) -> 2.7pF
- C32, C33: value (none) -> 6pF
- C34, C35: value (none) -> 5.2pF
- C36, C37: value (none) -> NC
- L1, L4: value (none) -> 39nH
- L2, L3: value (none) -> 120nH
- L5, L6: value (none) -> 27nH
- L7: value (none) -> 0R
Changed lines of the file:
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@@
 <attribute name="VALUE" x="33.274" y="23.7998" size="0.0254" layer="27" rot="R180"/>
 </element>
-<element name="C29" library="resistor" package="C0805" value="" x="81.2292" y="69.4944" smashed="yes" rot="R180">
+<element name="C29" library="resistor" package="C0805" value="2.7pF" x="81.2292" y="69.4944" smashed="yes" rot="R180">
 <attribute name="NAME" x="79.502" y="73.279" size="1.016" layer="25" font="vector" rot="R270"/>
 <attribute name="VALUE" x="82.1182" y="71.7804" size="1.27" layer="27" rot="R180"/>
 </element>
-<element name="L2" library="SparkFun-Coils" package="0805" value="" x="81.2292" y="67.6656" smashed="yes">
+<element name="L2" library="SparkFun-Coils" package="0805" value="120nH" x="81.2292" y="67.6656" smashed="yes">
 <attribute name="PROD_ID" value="NDUC-13076" x="82.4992" y="67.6656" size="1.778" layer="27" display="off"/>
 <attribute name="NAME" x="81.2292" y="66.1162" size="1.016" layer="25" font="vector" align="bottom-center"/>
 <attribute name="VALUE" x="81.2292" y="66.7766" size="0.6096" layer="27" font="vector" ratio="20" align="top-center"/>
 </element>
-<element name="C30" library="resistor" package="C0805" value="" x="84.7344" y="69.4944" smashed="yes" rot="R180">
+<element name="C30" library="resistor" package="C0805" value="2.7pF" x="84.7344" y="69.4944" smashed="yes" rot="R180">
 <attribute name="NAME" x="88.138" y="68.1482" size="1.016" layer="25" font="vector" rot="R90"/>
 <attribute name="VALUE" x="85.6234" y="71.7804" size="1.27" layer="27" rot="R180"/>
 </element>
-<element name="L3" library="SparkFun-Coils" package="0805" value="" x="84.582" y="67.6656" smashed="yes">
+<element name="L3" library="SparkFun-Coils" package="0805" value="120nH" x="84.582" y="67.6656" smashed="yes">
 <attribute name="PROD_ID" value="NDUC-13076" x="85.852" y="67.6656" size="1.778" layer="27" display="off"/>
 <attribute name="NAME" x="84.582" y="65.8114" size="1.016" layer="25" font="vector" align="bottom-center"/>
 <attribute name="VALUE" x="84.582" y="66.7766" size="0.6096" layer="27" font="vector" ratio="20" align="top-center"/>
 </element>
-<element name="L1" library="SparkFun-Coils" package="0805" value="" x="82.1436" y="72.2376" smashed="yes" rot="R270">
+<element name="L1" library="SparkFun-Coils" package="0805" value="39nH" x="82.1436" y="72.2376" smashed="yes" rot="R270">
 <attribute name="PROD_ID" value="NDUC-13076" x="82.1436" y="72.2376" size="1.778" layer="27" rot="R270" display="off"/>
 <attribute name="NAME" x="80.4418" y="72.2376" size="1.016" layer="25" font="vector" rot="R270" align="bottom-center"/>
 <attribute name="VALUE" x="81.2546" y="72.2376" size="0.6096" layer="27" font="vector" ratio="20" rot="R270" align="top-center"/>
 </element>
-<element name="L4" library="SparkFun-Coils" package="0805" value="" x="83.9724" y="72.2376" smashed="yes" rot="R270">
+<element name="L4" library="SparkFun-Coils" package="0805" value="39nH" x="83.9724" y="72.2376" smashed="yes" rot="R270">
 <attribute name="PROD_ID" value="NDUC-13076" x="83.9724" y="72.2376" size="1.778" layer="27" rot="R270" display="off"/>
 <attribute name="NAME" x="84.8614" y="72.5424" size="1.016" layer="25" font="vector" rot="R270" align="bottom-center"/>
 <attribute name="VALUE" x="83.0834" y="72.2376" size="0.6096" layer="27" font="vector" ratio="20" rot="R270" align="top-center"/>
 </element>
-<element name="C28" library="resistor" package="C0805" value="" x="84.1248" y="75.8952" smashed="yes" rot="R90">
+<element name="C28" library="resistor" package="C0805" value="7.5pF" x="84.1248" y="75.8952" smashed="yes" rot="R90">
 <attribute name="NAME" x="85.0646" y="75.3872" size="1.016" layer="25" font="vector"/>
 <attribute name="VALUE" x="86.4108" y="75.0062" size="1.27" layer="27" rot="R90"/>
 </element>
-<element name="C31" library="resistor" package="C0805" value="" x="81.9912" y="75.8952" smashed="yes" rot="R90">
+<element name="C31" library="resistor" package="C0805" value="7.5pF" x="81.9912" y="75.8952" smashed="yes" rot="R90">
 <attribute name="NAME" x="77.7494" y="75.692" size="1.016" layer="25" font="vector"/>
 <attribute name="VALUE" x="84.2772" y="75.0062" size="1.27" layer="27" rot="R90"/>
 </element>
-<element name="C32" library="resistor" package="C0805" value="" x="81.0768" y="79.0956" smashed="yes">
+<element name="C32" library="resistor" package="C0805" value="6pF" x="81.0768" y="79.0956" smashed="yes">
 <attribute name="NAME" x="78.9178" y="79.6036" size="1.016" layer="25" font="vector" rot="R180"/>
 <attribute name="VALUE" x="80.1878" y="76.8096" size="1.27" layer="27"/>
 </element>
-<element name="C33" library="resistor" package="C0805" value="" x="84.7344" y="79.0956" smashed="yes">
+<element name="C33" library="resistor" package="C0805" value="6pF" x="84.7344" y="79.0956" smashed="yes">
 <attribute name="NAME" x="86.5886" y="78.4352" size="1.016" layer="25" font="vector"/>
 <attribute name="VALUE" x="83.8454" y="76.8096" size="1.27" layer="27"/>
 </element>
-<element name="C34" library="resistor" package="C0805" value="" x="81.0768" y="81.0768" smashed="yes">
+<element name="C34" library="resistor" package="C0805" value="5.2pF" x="81.0768" y="81.0768" smashed="yes">
 <attribute name="NAME" x="79.2226" y="81.8896" size="1.016" layer="25" font="vector" rot="R180"/>
 <attribute name="VALUE" x="80.1878" y="78.7908" size="1.27" layer="27"/>
 </element>
-<element name="L5" library="SparkFun-Coils" package="0805" value="" x="84.8868" y="81.0768" smashed="yes" rot="R180">
+<element name="L5" library="SparkFun-Coils" package="0805" value="27nH" x="84.8868" y="81.0768" smashed="yes" rot="R180">
 <attribute name="PROD_ID" value="NDUC-13076" x="84.8868" y="81.0768" size="1.778" layer="27" rot="R180" display="off"/>
 <attribute name="NAME" x="87.4776" y="81.407" size="1.016" layer="25" font="vector" rot="R180" align="bottom-center"/>
 <attribute name="VALUE" x="84.8868" y="81.9658" size="0.6096" layer="27" font="vector" ratio="20" rot="R180" align="top-center"/>
 </element>
-<element name="L6" library="SparkFun-Coils" package="0805" value="" x="81.9912" y="83.9724" smashed="yes" rot="R90">
+<element name="L6" library="SparkFun-Coils" package="0805" value="27nH" x="81.9912" y="83.9724" smashed="yes" rot="R90">
 <attribute name="PROD_ID" value="NDUC-13076" x="81.9912" y="83.9724" size="1.778" layer="27" rot="R90" display="off"/>
 <attribute name="NAME" x="80.6196" y="84.1502" size="1.016" layer="25" font="vector" rot="R180" align="bottom-center"/>
 <attribute name="VALUE" x="82.8802" y="83.9724" size="0.6096" layer="27" font="vector" ratio="20" rot="R90" align="top-center"/>
 </element>
-<element name="C35" library="resistor" package="C0805" value="" x="83.9724" y="83.9724" smashed="yes" rot="R270">
+<element name="C35" library="resistor" package="C0805" value="5.2pF" x="83.9724" y="83.9724" smashed="yes" rot="R270">
 <attribute name="NAME" x="84.9122" y="83.1596" size="1.016" layer="25" font="vector"/>
 <attribute name="VALUE" x="81.6864" y="84.8614" size="1.27" layer="27" rot="R270"/>
 </element>
-<element name="C36" library="resistor" package="C0805" value="" x="84.8868" y="87.0204" smashed="yes" rot="R180">
+<element name="C36" library="resistor" package="C0805" value="NC" x="84.8868" y="87.0204" smashed="yes" rot="R180">
 <attribute name="NAME" x="82.7278" y="87.5284" size="1.016" layer="25" font="vector" rot="R180"/>
 <attribute name="VALUE" x="85.7758" y="89.3064" size="1.27" layer="27" rot="R180"/>
 </element>
-<element name="L7" library="SparkFun-Coils" package="0805" value="" x="84.0486" y="89.6874" smashed="yes" rot="R90">
+<element name="L7" library="SparkFun-Coils" package="0805" value="0R" x="84.0486" y="89.6874" smashed="yes" rot="R90">
 <attribute name="PROD_ID" value="NDUC-13076" x="84.0486" y="89.6874" size="1.778" layer="27" rot="R90" display="off"/>
 <attribute name="NAME" x="82.3722" y="89.5096" size="1.016" layer="25" font="vector" align="bottom-center"/>
 <attribute name="VALUE" x="84.9376" y="89.6874" size="0.6096" layer="27" font="vector" ratio="20" rot="R90" align="top-center"/>
 </element>
-<element name="C37" library="resistor" package="C0805" value="" x="84.8868" y="92.202" smashed="yes" rot="R180">
+<element name="C37" library="resistor" package="C0805" value="NC" x="84.8868" y="92.202" smashed="yes" rot="R180">
 <attribute name="NAME" x="83.693" y="93.5228" size="1.016" layer="25" font="vector"/>
 <attribute name="VALUE" x="85.7758" y="94.488" size="1.27" layer="27" rot="R180"/>

Commit message: Noticed that I forgot to apply the Calculations for Linear Voltage Regulators to eagle, fixed this
Parts:
- R53: value 5k1 -> 47k
- R54, R56, R58: value 47k -> 5k1
- R55: value 5k1 -> 33k
- R57: value 5k1 -> 8k2
Changed lines of the file:
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@@
 <attribute name="VALUE" x="67.1474" y="78.5148" size="1.016" layer="27" rot="R90"/>
 </element>
-<element name="R53" library="resistor" package="M0805" value="5k1" x="65.6844" y="89.916" smashed="yes">
+<element name="R53" library="resistor" package="M0805" value="47k" x="65.6844" y="89.916" smashed="yes">
 <attribute name="NAME" x="65.5828" y="90.932" size="1.016" layer="25" font="vector"/>
 <attribute name="VALUE" x="64.6684" y="87.63" size="1.27" layer="27"/>
 </element>
-<element name="R54" library="resistor" package="M0805" value="47k" x="64.9224" y="97.536" smashed="yes" rot="R90">
+<element name="R54" library="resistor" package="M0805" value="5k1" x="64.9224" y="97.536" smashed="yes" rot="R90">
 <attribute name="NAME" x="63.2968" y="96.2152" size="1.016" layer="25" font="vector" rot="R90"/>
 <attribute name="VALUE" x="67.2084" y="96.52" size="1.27" layer="27" rot="R90"/>
@@
 <attribute name="VALUE" x="24.0504" y="88.0262" size="1.016" layer="27" rot="R180"/>
 </element>
-<element name="R55" library="resistor" package="M0805" value="5k1" x="12.4968" y="86.106" smashed="yes" rot="R90">
+<element name="R55" library="resistor" package="M0805" value="33k" x="12.4968" y="86.106" smashed="yes" rot="R90">
 <attribute name="NAME" x="11.4808" y="85.09" size="1.016" layer="25" font="vector" rot="R90"/>
 <attribute name="VALUE" x="14.7828" y="85.09" size="1.27" layer="27" rot="R90"/>
 </element>
-<element name="R56" library="resistor" package="M0805" value="47k" x="4.8768" y="86.106" smashed="yes" rot="R180">
+<element name="R56" library="resistor" package="M0805" value="5k1" x="4.8768" y="86.106" smashed="yes" rot="R180">
 <attribute name="NAME" x="7.874" y="84.4804" size="1.016" layer="25" font="vector" rot="R180"/>
 <attribute name="VALUE" x="5.8928" y="88.392" size="1.27" layer="27" rot="R180"/>
@@
 <attribute name="VALUE" x="18.2592" y="67.9094" size="1.016" layer="27" rot="R180"/>
 </element>
-<element name="R57" library="resistor" package="M0805" value="5k1" x="26.67" y="73.6092" smashed="yes">
+<element name="R57" library="resistor" package="M0805" value="8k2" x="26.67" y="73.6092" smashed="yes">
 <attribute name="NAME" x="25.654" y="74.6252" size="1.016" layer="25" font="vector"/>
 <attribute name="VALUE" x="25.654" y="71.3232" size="1.27" layer="27"/>
 </element>
-<element name="R58" library="resistor" package="M0805" value="47k" x="26.3652" y="80.9244" smashed="yes" rot="R90">
+<element name="R58" library="resistor" package="M0805" value="5k1" x="26.3652" y="80.9244" smashed="yes" rot="R90">
 <attribute name="NAME" x="25.3492" y="79.9084" size="1.016" layer="25" font="vector" rot="R90"/>
 <attribute name="VALUE" x="28.6512" y="79.9084" size="1.27" layer="27" rot="R90"/>

Commit message: small schematic changes
Parts:
- R23, R24: value 220R -> 470R
Changed lines of the file:
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@@
 <layer number="25" name="tNames" color="7" fill="1" visible="yes" active="yes"/>
 <layer number="26" name="bNames" color="7" fill="1" visible="yes" active="yes"/>
-<layer number="27" name="tValues" color="7" fill="1" visible="no" active="yes"/>
+<layer number="27" name="tValues" color="7" fill="1" visible="yes" active="yes"/>
 <layer number="28" name="bValues" color="7" fill="1" visible="no" active="yes"/>
 <layer number="29" name="tStop" color="7" fill="3" visible="no" active="yes"/>
@@
 <attribute name="VALUE" x="25.5016" y="11.5316" size="1.27" layer="27" rot="R180"/>
 </element>
-<element name="R23" library="resistor" package="M0805" value="220R" x="28.194" y="9.2964" smashed="yes" rot="R180">
+<element name="R23" library="resistor" package="M0805" value="470R" x="28.194" y="9.2964" smashed="yes" rot="R180">
 <attribute name="NAME" x="25.654" y="10.3124" size="1.016" layer="25" font="vector"/>
 <attribute name="VALUE" x="29.21" y="11.5824" size="1.27" layer="27" rot="R180"/>
 </element>
-<element name="R24" library="resistor" package="M0805" value="220R" x="28.194" y="7.0104" smashed="yes" rot="R180">
+<element name="R24" library="resistor" package="M0805" value="470R" x="28.194" y="7.0104" smashed="yes" rot="R180">
 <attribute name="NAME" x="29.3624" y="5.842" size="1.016" layer="25" font="vector" rot="R180"/>
 <attribute name="VALUE" x="29.21" y="9.2964" size="1.27" layer="27" rot="R180"/>

Commit message: Accumulated Changes over a few weeks
Parts:
- R49: value 10k -> 3k9
- R51: value 120k -> 155k
- R53: value 47k -> 5k1
- R54: value 5k1 -> 39k
Changed lines of the file:
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@@
 <attribute name="VALUE" x="20.9644" y="45.9436" size="1.016" layer="27" rot="R180"/>
 </element>
-<element name="R49" library="resistor" package="M0805" value="10k" x="23.1648" y="46.7868" smashed="yes" rot="R90">
+<element name="R49" library="resistor" package="M0805" value="3k9" x="23.1648" y="46.7868" smashed="yes" rot="R90">
 <attribute name="NAME" x="22.1488" y="45.7708" size="1.016" layer="25" font="vector" rot="R90"/>
 <attribute name="VALUE" x="25.4508" y="45.7708" size="1.27" layer="27" rot="R90"/>
@@
 <attribute name="VALUE" x="29.6926" y="41.9862" size="1.27" layer="27" rot="R90"/>
 </element>
-<element name="R51" library="resistor" package="M0805" value="120k" x="1.524" y="43.7388" smashed="yes" rot="R90">
+<element name="R51" library="resistor" package="M0805" value="155k" x="1.524" y="43.7388" smashed="yes" rot="R90">
 <attribute name="NAME" x="2.3368" y="46.0756" size="1.016" layer="25" font="vector" rot="R90"/>
 <attribute name="VALUE" x="3.81" y="42.7228" size="1.27" layer="27" rot="R90"/>
@@
 <attribute name="VALUE" x="67.1474" y="78.5148" size="1.016" layer="27" rot="R90"/>
 </element>
-<element name="R53" library="resistor" package="M0805" value="47k" x="65.6844" y="89.916" smashed="yes">
+<element name="R53" library="resistor" package="M0805" value="5k1" x="65.6844" y="89.916" smashed="yes">
 <attribute name="NAME" x="65.5828" y="90.932" size="1.016" layer="25" font="vector"/>
 <attribute name="VALUE" x="64.6684" y="87.63" size="1.27" layer="27"/>
 </element>
-<element name="R54" library="resistor" package="M0805" value="5k1" x="64.9224" y="97.536" smashed="yes" rot="R90">
+<element name="R54" library="resistor" package="M0805" value="39k" x="64.9224" y="97.536" smashed="yes" rot="R90">
 <attribute name="NAME" x="63.2968" y="96.2152" size="1.016" layer="25" font="vector" rot="R90"/>
 <attribute name="VALUE" x="67.2084" y="96.52" size="1.27" layer="27" rot="R90"/>
